File: pico-power-switch.kicad/pico-power-switch.kicad_pcb (KiCad board)
At the start: 2 copper layers, 21 x 33.8 mm, 18 parts, among them J1 JST-PH2 Bat, J2 Pico Pin 1-13, J3 Pico Pin 40-28, J4 Alt-Bat, J5 Stemma-QT_Qwicc, Q1 AO3401A, Q2 AO3401A, SW1 SW_Push_SLIM, U1 74LVC2G74, U2 PCF8563T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

Commit message: Rev 1.0 (in production)
Parts:
- moved J5 27.1 mm to (109.1, 128.7), turned to 0 degrees
- moved J4 25.7 mm to (112.4, 102.8), turned to 90 degrees
- moved J1 23.8 mm to (111.1, 103.6), turned to 180 degrees
- moved SW1 20.1 mm to (110.9, 110.8), turned to 180 degrees
- moved R3 19.7 mm to (112.1, 124.8)
- moved R4 19.3 mm to (108.9, 124.8)
- moved Y1 13.6 mm to (104.2, 120.3), turned to -90 degrees
- moved U2 12.2 mm to (109.3, 121.5), turned to 0 degrees
- moved R2 9.69 mm to (105.0, 114.4)
- moved C2 7.86 mm to (112.1, 118.2), turned to 180 degrees
- moved C3 7.84 mm to (106.5, 118.1), turned to 180 degrees
- moved C1 3.28 mm to (105.5, 116.0), turned to -90 degrees
- moved U1 1.36 mm to (109.1, 114.9)
- moved R1 1.33 mm to (113.2, 115.9)
- moved Q1 0.28 mm to (104.0, 100.7)
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Routing:
- net /SDA: track 16.9 -> 33.8 mm, vias 0 -> 2
- net +3V3: track 18.3 -> 29.4 mm
- net /~{INT}: track 31.4 -> 24.4 mm, vias 0 -> 1
- net /PC_GATE: track 16.4 -> 12.9 mm, vias 2 -> 0
- net +BATT: track 39.4 -> 36.3 mm, vias 0 -> 2
- net GND: track 0.00 -> 2.80 mm, vias 0 -> 4
- net /SCL: track 26.4 -> 25.0 mm, vias 0 -> 2
- added copper zone on B.Cu, net GND
- added copper zone on F.Cu, net GND

Commit message: fixed schematic for power-connectors
Connections:
- J4 pad 1: GND -> +BATT
Changed lines of the file:
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@@
     (fp_line (start -1.27 -3.81) (end -1.27 0.635) (layer "B.Fab") (width 0.1))
     (pad "1" thru_hole rect (at 0 0 90) (size 1.7 1.7) (drill 1) (layers *.Cu *.Mask)
-      (net 2 "GND") (pinfunction "Pin_1") (pintype "passive"))
+      (net 1 "+BATT") (pinfunction "Pin_1") (pintype "passive"))
     (pad "2" thru_hole oval (at 0 -2.54 90) (size 1.7 1.7) (drill 1) (layers *.Cu *.Mask)
       (net 2 "GND") (pinfunction "Pin_2") (pintype "passive"))
